Commit message: gazebo launch file completed

File: ass1/ros2_ws/src/simmulator/description/iiwa7.xacro (robot description, xacro)
@@ -50,5 +50,5 @@
         <origin xyz="0 0 0" rpy="0 0 0"/>
         <geometry>
-          <mesh filename="package://simmulator/meshes/iiwa7/visual/link_0.stl"/>
+          <mesh filename="$(find simmulator)/meshes/iiwa7/visual/link_0.stl"/>
         </geometry>
         <material name="Grey"/>
@@ -57,5 +57,5 @@
         <origin xyz="0 0 0" rpy="0 0 0"/>
         <geometry>
-          <mesh filename="package://simmulator/meshes/iiwa7/collision/link_0.stl"/>
+          <mesh filename="$(find simmulator)/meshes/iiwa7/collision/link_0.stl"/>
         </geometry>
         <material name="Grey"/>
@@ -92,5 +92,5 @@
         <origin xyz="0 0 0.0075" rpy="0 0 0"/>
         <geometry>
-          <mesh filename="package://simmulator/meshes/iiwa7/visual/link_1.stl"/>
+          <mesh filename="$(find simmulator)/meshes/iiwa7/visual/link_1.stl"/>
         </geometry>
         <material name="Orange"/>
@@ -99,5 +99,5 @@
         <origin xyz="0 0 0.0075" rpy="0 0 0"/>
         <geometry>
-          <mesh filename="package://simmulator/meshes/iiwa7/collision/link_1.stl"/>
+          <mesh filename="$(find simmulator)/meshes/iiwa7/collision/link_1.stl"/>
         </geometry>
         <material name="Orange"/>
@@ -127,5 +127,5 @@
         <origin xyz="0 0 0" rpy="0 0 0"/>
         <geometry>
-          <mesh filename="package://simmulator/meshes/iiwa7/visual/link_2.stl"/>
+          <mesh filename="$(find simmulator)/meshes/iiwa7/visual/link_2.stl"/>
         </geometry>
         <material name="Orange"/>
@@ -134,5 +134,5 @@
         <origin xyz="0 0 0" rpy="0 0 0"/>
         <geometry>
-          <mesh filename="package://simmulator/meshes/iiwa7/collision/link_2.stl"/>
+          <mesh filename="$(find simmulator)/meshes/iiwa7/collision/link_2.stl"/>
         </geometry>
         <material name="Orange"/>
