Commit message: update

File: ass3/ros2_ws_2/scr/owl/urdf/robot.urdf (robot description, URDF)
Before this commit: robot owl_robot, 10 links, 9 joints
Links:
- link base_link: geometry collision mesh filename=package://owl/meshes/base_link.STL; visual mesh filename=package://owl/meshes/base_link.STL
- link elbow_link: geometry collision mesh filename=package://owl/meshes/elbow_link.STL; visual mesh filename=package://owl/meshes/elbow_link.STL
- link end_effector_link: geometry collision mesh filename=package://owl/meshes/end_effector_link.STL; visual mesh filename=package://owl/meshes/end_effector_link.STL
- link link1: geometry collision mesh filename=package://owl/meshes/link1.STL; visual mesh filename=package://owl/meshes/link1.STL
- link link2: geometry collision mesh filename=package://owl/meshes/link2.STL; visual mesh filename=package://owl/meshes/link2.STL
- link shoulder_link: geometry collision mesh filename=package://owl/meshes/shoulder_link.STL; visual mesh filename=package://owl/meshes/shoulder_link.STL
- link w2w3_link: geometry collision mesh filename=package://owl/meshes/w2w3_link.STL; visual mesh filename=package://owl/meshes/w2w3_link.STL

File: ass3/ros2_ws_2/scr/owl/urdf/robot.xacro (robot description, xacro)
@@ -31,5 +31,5 @@
       <geometry>
         <mesh
-          filename="package://owl_robot_description/meshes/base_link.STL" />
+          filename="package://owl/meshes/base_link.STL" />
       </geometry>
       <material
@@ -45,5 +45,5 @@
       <geometry>
         <mesh
-          filename="package://owl_robot_description/meshes/base_link.STL" />
+          filename="package://owl/meshes/base_link.STL" />
       </geometry>
     </collision>
@@ -71,19 +71,19 @@
       <geometry>
         <mesh
-          filename="package://owl_robot_description/meshes/shoulder_link.STL" />
-      </geometry>
-      <material
-        name="">
-        <color
-          rgba="0.79216 0.81961 0.93333 1" />
-      </material>
-    </visual>
-    <collision>
-      <origin
-        xyz="0 0 0"
-        rpy="0 0 0" />
-      <geometry>
-        <mesh
-          filename="package://owl_robot_description/meshes/shoulder_link.STL" />
+          filename="package://owl/meshes/shoulder_link.STL" />
+      </geometry>
+      <material
+        name="">
+        <color
+          rgba="0.79216 0.81961 0.93333 1" />
+      </material>
+    </visual>
+    <collision>
+      <origin
+        xyz="0 0 0"
+        rpy="0 0 0" />
+      <geometry>
+        <mesh
+          filename="package://owl/meshes/shoulder_link.STL" />
       </geometry>
     </collision>
@@ -125,19 +125,19 @@
       <geometry>
         <mesh
-          filename="package://owl_robot_description/meshes/link1.STL" />
-      </geometry>
-      <material
-        name="">
-        <color
-          rgba="0.79216 0.81961 0.93333 1" />
-      </material>
-    </visual>
-    <collision>
-      <origin
-        xyz="0 0 0"
-        rpy="0 0 0" />
-      <geometry>
-        <mesh
-          filename="package://owl_robot_description/meshes/link1.STL" />
+          filename="package://owl/meshes/link1.STL" />
+      </geometry>
+      <material
+        name="">
+        <color
+          rgba="0.79216 0.81961 0.93333 1" />
+      </material>
+    </visual>
+    <collision>
+      <origin
+        xyz="0 0 0"
+        rpy="0 0 0" />
+      <geometry>
+        <mesh
+          filename="package://owl/meshes/link1.STL" />
       </geometry>
     </collision>
@@ -179,19 +179,19 @@
       <geometry>
         <mesh
-          filename="package://owl_robot_description/meshes/elbow_link.STL" />
-      </geometry>
-      <material
-        name="">
-        <color
-          rgba="0.79216 0.81961 0.93333 1" />
-      </material>
-    </visual>
-    <collision>
-      <origin
-        xyz="0 0 0"
-        rpy="0 0 0" />
-      <geometry>
-        <mesh
-          filename="package://owl_robot_description/meshes/elbow_link.STL" />
+          filename="package://owl/meshes/elbow_link.STL" />
+      </geometry>
+      <material
+        name="">
+        <color
+          rgba="0.79216 0.81961 0.93333 1" />
+      </material>
+    </visual>
+    <collision>
+      <origin
+        xyz="0 0 0"
+        rpy="0 0 0" />
+      <geometry>
+        <mesh
+          filename="package://owl/meshes/elbow_link.STL" />
       </geometry>
     </collision>
@@ -233,19 +233,19 @@
       <geometry>
         <mesh
-          filename="package://owl_robot_description/meshes/link2.STL" />
-      </geometry>
-      <material
-        name="">
-        <color
-          rgba="0.79216 0.81961 0.93333 1" />
-      </material>
-    </visual>
-    <collision>
-      <origin
-        xyz="0 0 0"
-        rpy="0 0 0" />
-      <geometry>
-        <mesh
-          filename="package://owl_robot_description/meshes/link2.STL" />
+          filename="package://owl/meshes/link2.STL" />
+      </geometry>
+      <material
+        name="">
+        <color
+          rgba="0.79216 0.81961 0.93333 1" />
+      </material>
+    </visual>
+    <collision>
+      <origin
+        xyz="0 0 0"
+        rpy="0 0 0" />
+      <geometry>
+        <mesh
+          filename="package://owl/meshes/link2.STL" />
       </geometry>
     </collision>
@@ -287,19 +287,19 @@
       <geometry>
         <mesh
-          filename="package://owl_robot_description/meshes/w2w3_link.STL" />
-      </geometry>
-      <material
-        name="">
-        <color
-          rgba="0.79216 0.81961 0.93333 1" />
-      </material>
-    </visual>
-    <collision>
-      <origin
-        xyz="0 0 0"
-        rpy="0 0 0" />
-      <geometry>
-        <mesh
-          filename="package://owl_robot_description/meshes/w2w3_link.STL" />
+          filename="package://owl/meshes/w2w3_link.STL" />
+      </geometry>
+      <material
+        name="">
+        <color
+          rgba="0.79216 0.81961 0.93333 1" />
+      </material>
+    </visual>
+    <collision>
+      <origin
+        xyz="0 0 0"
+        rpy="0 0 0" />
+      <geometry>
+        <mesh
+          filename="package://owl/meshes/w2w3_link.STL" />
       </geometry>
     </collision>
@@ -341,19 +341,19 @@
       <geometry>
         <mesh
-          filename="package://owl_robot_description/meshes/end_effector_link.STL" />
-      </geometry>
-      <material
-        name="">
-        <color
-          rgba="0.79216 0.81961 0.93333 1" />
-      </material>
-    </visual>
-    <collision>
-      <origin
-        xyz="0 0 0"
-        rpy="0 0 0" />
-      <geometry>
-        <mesh
-          filename="package://owl_robot_description/meshes/end_effector_link.STL" />
+          filename="package://owl/meshes/end_effector_link.STL" />
+      </geometry>
+      <material
+        name="">
+        <color
+          rgba="0.79216 0.81961 0.93333 1" />
+      </material>
+    </visual>
+    <collision>
+      <origin
+        xyz="0 0 0"
+        rpy="0 0 0" />
+      <geometry>
+        <mesh
+          filename="package://owl/meshes/end_effector_link.STL" />
       </geometry>
     </collision>

File: ass3/ros2_ws_2/scr/owl/urdf/robot_active.urdf (robot description, URDF)
Before this commit: robot owl_robot, 10 links, 9 joints
Links:
- link base_link: geometry collision mesh filename=package://owl/meshes/base_link.STL; visual mesh filename=package://owl/meshes/base_link.STL
- link elbow_link: geometry collision mesh filename=package://owl/meshes/elbow_link.STL; visual mesh filename=package://owl/meshes/elbow_link.STL
- link end_effector_link: geometry collision mesh filename=package://owl/meshes/end_effector_link.STL; visual mesh filename=package://owl/meshes/end_effector_link.STL
- link link1: geometry collision mesh filename=package://owl/meshes/link1.STL; visual mesh filename=package://owl/meshes/link1.STL
- link link2: geometry collision mesh filename=package://owl/meshes/link2.STL; visual mesh filename=package://owl/meshes/link2.STL
- link shoulder_link: geometry collision mesh filename=package://owl/meshes/shoulder_link.STL; visual mesh filename=package://owl/meshes/shoulder_link.STL
- link w2w3_link: geometry collision mesh filename=package://owl/meshes/w2w3_link.STL; visual mesh filename=package://owl/meshes/w2w3_link.STL
